File: kicad/stm32l053c.sch (KiCad schematic (older format))
At the start: 39 parts, among them J1 GND, J10 3V3, J11 I2C, J2 GND, J3 TX, J4 GND, J8 RX, P1 SWD, U1 AP2112, U2 STM32L053C8_LQFP48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

Commit message: Start of pin assignment
Parts:
- removed A0: A0, Pin_Headers:Pin_Header_Straight_1x01_Pitch2.54mm, symbol stm32l053c-rescue:CONN_01X01
- removed A1: A1, Pin_Headers:Pin_Header_Straight_1x01_Pitch2.54mm, symbol stm32l053c-rescue:CONN_01X01
- removed A2: A2, Pin_Headers:Pin_Header_Straight_1x01_Pitch2.54mm, symbol stm32l053c-rescue:CONN_01X01
- removed C4: 10uF, Capacitors_SMD:C_0805_HandSoldering, symbol stm32l053c-rescue:C
- removed D2: D_Schottky, theapi:D_SOD-323_HandSoldering, symbol stm32l053c-rescue:D_Schottky
- removed J1, J2, J4: GND, Pin_Headers:Pin_Header_Straight_1x01_Pitch2.54mm, symbol stm32l053c-rescue:CONN_01X01
- removed J10: 3V3, Pin_Headers:Pin_Header_Straight_1x01_Pitch2.54mm, symbol stm32l053c-rescue:CONN_01X01
- removed J11: I2C, Pin_Headers:Pin_Header_Straight_1x04_Pitch2.54mm, symbol stm32l053c-rescue:CONN_01X04
- removed J3: TX, Pin_Headers:Pin_Header_Straight_1x01_Pitch2.54mm, symbol stm32l053c-rescue:CONN_01X01
- removed J8: RX, Pin_Headers:Pin_Header_Straight_1x01_Pitch2.54mm, symbol stm32l053c-rescue:CONN_01X01
- removed R6: 300K, Resistors_SMD:R_0805_HandSoldering, symbol stm32l053c-rescue:R
- removed R7: 100K, Resistors_SMD:R_0805_HandSoldering, symbol stm32l053c-rescue:R
- removed SC1: Solar_Cells, Pin_Headers:Pin_Header_Straight_1x02_Pitch2.54mm, symbol stm32l053c-rescue:Solar_Cells
- removed U1: AP2112, TO_SOT_Packages_SMD:SOT-23-5_HandSoldering, symbol theapi_voltage_regulators:AP2112
- added J?: Motion, symbol Connector:Conn_01x03_Female
- added Q?: Q_NMOS_GSD, symbol Device:Q_NMOS_GSD
- added R?: 1K, symbol Device:R
- added U?: MCP1703A-3302_SOT223, Package_TO_SOT_SMD:SOT-223-3_TabPin2, symbol Regulator_Linear:MCP1703A-3302_SOT223
Connections:
- net labels added: DOOR, MOTION, PUMP, SENSOR_GND, WATER_TEMP
- net labels removed: USART1_RX, USART1_TX
- wire segments 82 -> 72
- no-connect marks 23 -> 13
Other:
- note added: "Max 16v"
- note removed: "Max 6v"
- moved on the sheet: C1, C2, C3, C5, C6, C9, R4, R8, R9, U2

Commit message: Schematic
Parts:
- added D2: LED_CRGB, Connector_JST:JST_XH_B04B-XH-A_1x04_P2.50mm_Vertical, symbol Device:LED_CRGB
- added J1: Water_Level, Connector_JST:JST_XH_B02B-XH-A_1x02_P2.50mm_Vertical, symbol Connector:Conn_01x02_Female
- added J3: Door, Connector_JST:JST_XH_B02B-XH-A_1x02_P2.50mm_Vertical, symbol Connector:Conn_01x02_Female
- added J4: Door_Led, Connector_JST:JST_XH_B02B-XH-A_1x02_P2.50mm_Vertical, symbol Connector:Conn_01x02_Female
- added J5: AIN3, Connector_JST:JST_XH_B02B-XH-A_1x02_P2.50mm_Vertical, symbol Connector:Conn_01x02_Female
- added J6: Pump, Connector_PinHeader_2.54mm:PinHeader_1x01_P2.54mm_Vertical, symbol Connector:Conn_01x01_Female
- added R11, R12, R7: 100K, Resistor_SMD:R_0805_2012Metric_Pad1.15x1.40mm_HandSolder, symbol Device:R
- added R14: 620K, Resistors_SMD:R_0805_HandSoldering, symbol stm32l053c-rescue:R
- added R15: 100K, Resistors_SMD:R_0805_HandSoldering, symbol stm32l053c-rescue:R
- added R16, R17, R18: 820, Resistor_SMD:R_0805_2012Metric_Pad1.15x1.40mm_HandSolder, symbol Device:R
- added R6: 10K, Resistor_SMD:R_0603_1608Metric_Pad1.05x0.95mm_HandSolder, symbol Device:R
- added TH1: Thermistor_NTC, Connector_JST:JST_XH_B02B-XH-A_1x02_P2.50mm_Vertical, symbol Device:Thermistor_NTC
- J2: renamed from J?; footprint (none) -> Connector_JST:JST_XH_B03B-XH-A_1x03_P2.50mm_Vertical
- Q1: renamed from Q?; footprint (none) -> Package_TO_SOT_SMD:SOT-23_Handsoldering
- R10, R2, R3, R4: footprint Resistors_SMD:R_0805_HandSoldering -> Resistor_SMD:R_0603_1608Metric_Pad1.05x0.95mm_HandSolder
- R13: renamed from R?; footprint (none) -> Resistor_SMD:R_0603_1608Metric_Pad1.05x0.95mm_HandSolder
- R8: value 100K -> 620K
- R9: footprint Resistors_SMD:R_0805_HandSoldering -> Resistor_SMD:R_0805_2012Metric_Pad1.15x1.40mm_HandSolder
- gave numbers to parts that had none: 1
Connections:
- net labels added: DOOR_LED, LED_BLUE, LED_GREEN, LED_RED, SENSOR_PWR, WATER_LEVEL
- net labels removed: SENSOR_GND
- wire segments 72 -> 92
- no-connect marks 13 -> 18
Other:
- moved on the sheet: C7, J2, Q1, R10, R13, R2, R3, U3

Commit message: Start of layout
Parts:
- removed BT1: Battery, theapi:BatteryBoxAndPins, symbol stm32l053c-rescue:Battery
- removed R5: R_Shunt, theapi:SHUNT_1210_HandSoldering, symbol stm32l053c-rescue:R_Shunt
- added H1, H2, H3, H4: MountingHole_Pad, MountingHole:MountingHole_3.2mm_M3_Pad, symbol Mechanical:MountingHole_Pad
- added J7: BATTERY, Connector_JST:JST_XH_B02B-XH-A_1x02_P2.50mm_Vertical, symbol Connector:Conn_01x02_Male
- added R5: 0.01R, Connector_JST:JST_XH_B02B-XH-A_1x02_P2.50mm_Vertical, symbol Device:R
- J5: footprint Connector_JST:JST_XH_B02B-XH-A_1x02_P2.50mm_Vertical -> Connector_PinHeader_2.54mm:PinHeader_1x02_P2.54mm_Vertical
- R1, R14, R15, R8: footprint Resistors_SMD:R_0805_HandSoldering -> Resistor_SMD:R_0805_2012Metric_Pad1.15x1.40mm_HandSolder
- U3: footprint Housings_SSOP:TSSOP-10_3x3mm_Pitch0.5mm -> Package_SO:TSSOP-10_3x3mm_P0.5mm
Connections:
- net labels added: +BATT
- wire segments 92 -> 94
Other:
- note added: "Shunt on low side of the battery"
- moved on the sheet: R8, R9
Changed lines of the file:
@@
 F 0 "R1" V 4280 2700 50  0000 C CNN
 F 1 "820" V 4200 2700 50  0000 C CNN
-F 2 "Resistors_SMD:R_0805_HandSoldering" V 4130 2700 50  0001 C CNN
+F 2 "Resistor_SMD:R_0805_2012Metric_Pad1.15x1.40mm_HandSolder" V 4130 2700 50  0001 C CNN
 F 3 "" H 4200 2700 50  0000 C CNN
 	1    4200 2700
@@
 F 0 "U3" H 2250 5475 50  0000 L CNN
 F 1 "ADS1015" H 3100 5475 50  0000 L CNN
-F 2 "Housings_SSOP:TSSOP-10_3x3mm_Pitch0.5mm" H 2800 4975 50  0001 C CNN
+F 2 "Package_SO:TSSOP-10_3x3mm_P0.5mm" H 2800 4975 50  0001 C CNN
 F 3 "" H 1950 5425 50  0001 C CNN
 	1    2850 5025
@@
 Text Notes 3175 2525 0    98   ~ 20
 Debug
-$Comp
-L stm32l053c-rescue:Battery BT1
-U 1 1 59319095
-P 1275 1325
-F 0 "BT1" H 1375 1425 50  0000 L CNN
-F 1 "Battery" H 1375 1325 50  0000 L CNN
-F 2 "theapi:BatteryBoxAndPins" V 1275 1385 50  0001 C CNN
-F 3 "" V 1275 1385 50  0001 C CNN
-	1    1275 1325
-	1    0    0    -1
-$EndComp
-$Comp
-L power:Earth #PWR028
-U 1 1 593290F6
-P 1275 1925
-F 0 "#PWR028" H 1275 1675 50  0001 C CNN
-F 1 "Earth" H 1275 1775 50  0001 C CNN
-F 2 "" H 1275 1925 50  0000 C CNN
-F 3 "" H 1275 1925 50  0000 C CNN
-	1    1275 1925
-	1    0    0    -1
-$EndComp
 Text GLabel 10625 3800 2    60   Input ~ 0
 RFM_RST
@@
 L stm32l053c-rescue:R R9
 U 1 1 59356DA1
-P 2150 1825
-F 0 "R9" V 2230 1825 50  0000 C CNN
-F 1 "100K" V 2150 1825 50  0000 C CNN
-F 2 "Resistor_SMD:R_0805_2012Metric_Pad1.15x1.40mm_HandSolder" V 2080 1825 50  0001 C CNN
-F 3 "" H 2150 1825 50  0001 C CNN
-	1    2150 1825
+P 2400 1825
+F 0 "R9" V 2480 1825 50  0000 C CNN
+F 1 "100K" V 2400 1825 50  0000 C CNN
+F 2 "Resistor_SMD:R_0805_2012Metric_Pad1.15x1.40mm_HandSolder" V 2330 1825 50  0001 C CNN
+F 3 "" H 2400 1825 50  0001 C CNN
+	1    2400 1825
 	1    0    0    -1
 $EndComp
@@
 L stm32l053c-rescue:R R8
 U 1 1 59356E2E
-P 2350 1625
-F 0 "R8" V 2430 1625 50  0000 C CNN
-F 1 "620K" V 2350 1625 50  0000 C CNN
-F 2 "Resistors_SMD:R_0805_HandSoldering" V 2280 1625 50  0001 C CNN
-F 3 "" H 2350 1625 50  0001 C CNN
-	1    2350 1625
+P 2600 1625
+F 0 "R8" V 2680 1625 50  0000 C CNN
+F 1 "620K" V 2600 1625 50  0000 C CNN
+F 2 "Resistor_SMD:R_0805_2012Metric_Pad1.15x1.40mm_HandSolder" V 2530 1625 50  0001 C CNN
+F 3 "" H 2600 1625 50  0001 C CNN
+	1    2600 1625
 	0    1    1    0
 $EndComp
@@
 L power:Earth #PWR030
 U 1 1 59357323
-P 2150 1975
-F 0 "#PWR030" H 2150 1725 50  0001 C CNN
-F 1 "Earth" H 2150 1825 50  0001 C CNN
-F 2 "" H 2150 1975 50  0000 C CNN
-F 3 "" H 2150 1975 50  0000 C CNN
-	1    2150 1975
+P 2400 1975
+F 0 "#PWR030" H 2400 1725 50  0001 C CNN
+F 1 "Earth" H 2400 1825 50  0001 C CNN
+F 2 "" H 2400 1975 50  0000 C CNN
+F 3 "" H 2400 1975 50  0000 C CNN
+	1    2400 1975
 	-1   0    0    -1
 $EndComp
@@
 Text Label 1900 5225 0    60   ~ 0
 AIN3
-$Comp
-L stm32l053c-rescue:R_Shunt R5
-U 1 1 593784A2
-P 1275 1725
-F 0 "R5" V 1100 1725 50  0000 C CNN
-F 1 "R_Shunt" V 1175 1725 50  0000 C CNN
-F 2 "theapi:SHUNT_1210_HandSoldering" V 1205 1725 50  0001 C CNN
-F 3 "" H 1275 1725 50  0001 C CNN
-	1    1275 1725
-	1    0    0    -1
-$EndComp
 Wire Wire Line
 	9225 6050 9225 6200
@@
 Connection ~ 4150 4325
 Wire Wire Line
-	1900 1625 2150 1625
-Wire Wire Line
-	2150 1625 2150 1675
-Text Label 1900 1625 0    60   ~ 0
+	2150 1625 2400 1625
+Wire Wire Line
+	2400 1625 2400 1675
+Text Label 2150 1625 0    60   ~ 0
 AIN2
-Connection ~ 2150 1625
-Text Label 1700 1825 2    60   ~ 0
+Connection ~ 2400 1625
+Text Label 1575 1775 2    60   ~ 0
 AIN0
-Text Label 1700 1625 2    60   ~ 0
+Text Label 1575 1475 2    60   ~ 0
 AIN1
-Text Label 1825 1125 0    60   ~ 0
+Text Label 2975 1300 0    60   ~ 0
 BATT
 Wire Wire Line
@@
 	4150 4325 4350 4325
 Wire Wire Line
-	2150 1625 2200 1625
+	2400 1625 2450 1625
 NoConn ~ 3400 7025
 NoConn ~ 4350 6925
@@
 Wire Wire Line
 	4125 1475 4525 1475
-Wire Wire Line
-	1425 1625 1700 1625
-Wire Wire Line
-	1425 1825 1700 1825
-Connection ~ 3200 1475
-Wire Wire Line
-	1275 1125 2500 1125
-Wire Wire Line
-	3200 1125 3200 1475
-Wire Wire Line
-	2500 1125 2500 1625
-Connection ~ 2500 1125
-Wire Wire Line
-	2500 1125 3200 1125
 Wire Notes Line
 	5075 2125 5075 725
@@
 F 0 "R15" V 1730 5375 50  0000 C CNN
 F 1 "100K" V 1650 5375 50  0000 C CNN
-F 2 "Resistors_SMD:R_0805_HandSoldering" V 1580 5375 50  0001 C CNN
+F 2 "Resistor_SMD:R_0805_2012Metric_Pad1.15x1.40mm_HandSolder" V 1580 5375 50  0001 C CNN
 F 3 "" H 1650 5375 50  0001 C CNN
 	1    1650 5375
@@
 F 0 "R14" V 1580 5225 50  0000 C CNN
 F 1 "620K" V 1500 5225 50  0000 C CNN
-F 2 "Resistors_SMD:R_0805_HandSoldering" V 1430 5225 50  0001 C CNN
+F 2 "Resistor_SMD:R_0805_2012Metric_Pad1.15x1.40mm_HandSolder" V 1430 5225 50  0001 C CNN
 F 3 "" H 1500 5225 50  0001 C CNN
 	1    1500 5225
@@
 F 0 "J5" H 1044 5000 50  0000 C CNN
 F 1 "AIN3" H 1044 5091 50  0000 C CNN
-F 2 "Connector_JST:JST_XH_B02B-XH-A_1x02_P2.50mm_Vertical" H 1150 5325 50  0001 C CNN
+F 2 "Connector_PinHeader_2.54mm:PinHeader_1x02_P2.54mm_Vertical" H 1150 5325 50  0001 C CNN
 F 3 "~" H 1150 5325 50  0001 C CNN
 	1    1150 5325
@@
 Wire Wire Line
 	5875 5775 5900 5775
+$Comp
+L Device:R R5
+U 1 1 5C243ACF
+P 1275 1625
+F 0 "R5" V 1200 1625 50  0000 C CNN
+F 1 "0.01R" V 1350 1625 50  0000 C CNN
+F 2 "Connector_JST:JST_XH_B02B-XH-A_1x02_P2.50mm_Vertical" V 1205 1625 50  0001 C CNN
+F 3 "~" H 1275 1625 50  0001 C CNN
+	1    1275 1625
+	-1   0    0    1
+$EndComp
+$Comp
+L power:+BATT #PWR0101
+U 1 1 5C268BEB
+P 2200 1175
+F 0 "#PWR0101" H 2200 1025 50  0001 C CNN
+F 1 "+BATT" H 2215 1348 50  0000 C CNN
+F 2 "" H 2200 1175 50  0001 C CNN
+F 3 "" H 2200 1175 50  0001 C CNN
+	1    2200 1175
+	1    0    0    -1
+$EndComp
+Wire Wire Line
+	3200 1300 3200 1475
+Connection ~ 3200 1475
+Wire Wire Line
+	2750 1625 2925 1625
+Wire Wire Line
+	2925 1625 2925 1300
+Wire Wire Line
+	2925 1300 3200 1300
+Wire Wire Line
+	1275 1775 1575 1775
+Wire Wire Line
+	1275 1475 1575 1475
+$Comp
+L Connector:Conn_01x02_Male J7
+U 1 1 5C27E7B1
+P 2000 1175
+F 0 "J7" H 1972 1055 50  0000 R CNN
+F 1 "BATTERY" H 2075 1250 50  0000 R CNN
+F 2 "Connector_JST:JST_XH_B02B-XH-A_1x02_P2.50mm_Vertical" H 2000 1175 50  0001 C CNN
+F 3 "~" H 2000 1175 50  0001 C CNN
+	1    2000 1175
+	1    0    0    -1
+$EndComp
+$Comp
+L power:Earth #PWR038
+U 1 1 5C2872F9
+P 2200 1275
+F 0 "#PWR038" H 2200 1025 50  0001 C CNN
+F 1 "Earth" H 2200 1125 50  0001 C CNN
+F 2 "" H 2200 1275 50  0000 C CNN
+F 3 "" H 2200 1275 50  0000 C CNN
+	1    2200 1275
+	1    0    0    -1
+$EndComp
+Wire Wire Line
+	2200 1175 2925 1175
+Wire Wire Line
+	2925 1175 2925 1300
+Connection ~ 2200 1175
+Connection ~ 2925 1300
+$Comp
+L Mechanical:MountingHole_Pad H1
+U 1 1 5C28F0A3
+P 8825 625
+F 0 "H1" H 8925 676 50  0000 L CNN
+F 1 "MountingHole_Pad" H 8925 585 50  0000 L CNN
+F 2 "MountingHole:MountingHole_3.2mm_M3_Pad" H 8825 625 50  0001 C CNN
+F 3 "~" H 8825 625 50  0001 C CNN
+	1    8825 625
+	1    0    0    -1
+$EndComp
+$Comp
+L power:Earth #PWR040
+U 1 1 5C28F4C4
+P 8825 725
+F 0 "#PWR040" H 8825 475 50  0001 C CNN
+F 1 "Earth" H 8825 575 50  0001 C CNN
+F 2 "" H 8825 725 50  0000 C CNN
+F 3 "" H 8825 725 50  0000 C CNN
+	1    8825 725
+	1    0    0    -1
+$EndComp
+$Comp
+L Mechanical:MountingHole_Pad H3
+U 1 1 5C28F591
+P 8825 1050
+F 0 "H3" H 8925 1101 50  0000 L CNN
+F 1 "MountingHole_Pad" H 8925 1010 50  0000 L CNN
+F 2 "MountingHole:MountingHole_3.2mm_M3_Pad" H 8825 1050 50  0001 C CNN
+F 3 "~" H 8825 1050 50  0001 C CNN
+	1    8825 1050
+	1    0    0    -1
+$EndComp
+$Comp
+L power:Earth #PWR042
+U 1 1 5C28F598
+P 8825 1150
+F 0 "#PWR042" H 8825 900 50  0001 C CNN
+F 1 "Earth" H 8825 1000 50  0001 C CNN
+F 2 "" H 8825 1150 50  0000 C CNN
+F 3 "" H 8825 1150 50  0000 C CNN
+	1    8825 1150
+	1    0    0    -1
+$EndComp
+$Comp
+L Mechanical:MountingHole_Pad H2
+U 1 1 5C294F15
+P 8525 850
+F 0 "H2" H 8625 901 50  0000 L CNN
+F 1 "MountingHole_Pad" H 8625 810 50  0000 L CNN
+F 2 "MountingHole:MountingHole_3.2mm_M3_Pad" H 8525 850 50  0001 C CNN
+F 3 "~" H 8525 850 50  0001 C CNN
+	1    8525 850
+	1    0    0    -1
+$EndComp
+$Comp
+L power:Earth #PWR041
+U 1 1 5C294F1C
+P 8525 950
+F 0 "#PWR041" H 8525 700 50  0001 C CNN
+F 1 "Earth" H 8525 800 50  0001 C CNN
+F 2 "" H 8525 950 50  0000 C CNN
+F 3 "" H 8525 950 50  0000 C CNN
+	1    8525 950
+	1    0    0    -1
+$EndComp
+$Comp
+L Mechanical:MountingHole_Pad H4
+U 1 1 5C294F22
+P 8525 1275
+F 0 "H4" H 8625 1326 50  0000 L CNN
+F 1 "MountingHole_Pad" H 8625 1235 50  0000 L CNN
+F 2 "MountingHole:MountingHole_3.2mm_M3_Pad" H 8525 1275 50  0001 C CNN
+F 3 "~" H 8525 1275 50  0001 C CNN
+	1    8525 1275
+	1    0    0    -1
+$EndComp
+$Comp
+L power:Earth #PWR043
+U 1 1 5C294F29
+P 8525 1375
+F 0 "#PWR043" H 8525 1125 50  0001 C CNN
+F 1 "Earth" H 8525 1225 50  0001 C CNN
+F 2 "" H 8525 1375 50  0000 C CNN
+F 3 "" H 8525 1375 50  0000 C CNN
+	1    8525 1375
+	1    0    0    -1
+$EndComp
+Text Notes 1075 1875 0    31   Italic 0
+Shunt on low side of the battery
 $EndSCHEMATC
