File: kicad/stm32l053c.sch (KiCad schematic (older format))
At the start: 57 parts, among them J1 Water_Level, J2 Motion, J3 Door, J4 Door_Led, J6 Pump, J7 BATTERY, P1 SWD, Q1 Q_NMOS_GSD, Q2 Q_PMOS_GSD, SW1 SW_Push_SPDT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

Commit message: Cap value
Parts:
- C7: value 10uF -> 0.1UF
Changed lines of the file:
@@
 P 3800 4375
 F 0 "C7" H 3825 4475 50  0000 L CNN
-F 1 "10uF" H 3825 4275 50  0000 L CNN
+F 1 "0.1UF" H 3825 4275 50  0000 L CNN
 F 2 "Capacitor_SMD:C_0805_2012Metric_Pad1.15x1.40mm_HandSolder" H 3838 4225 50  0001 C CNN
 F 3 "" H 3800 4375 50  0001 C CNN
