File: kicad/stm32l053c.kicad_pcb (KiCad board)
At the start: 2 copper layers, 90 x 70 mm, 60 parts, among them J1 Water_Level, J2 Motion, J3 Door, J4 Door_Led, J6 Pump, J7 BATTERY, P1 SWD, Q1 Q_NMOS_GSD, Q2 Q_PMOS_GSD, SW1 SW_Push_SPDT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

Commit message: Ordered from JLCPCB
Other:
- board text added: "1"
Changed lines of the file:
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@@
-(kicad_pcb (version 20171130) (host pcbnew "(5.0.0-3-g5ebb6b6)")
+(kicad_pcb (version 20171130) (host pcbnew 5.0.2-bee76a0~70~ubuntu16.04.1)
   (general
     (thickness 1.6)
-    (drawings 45)
+    (drawings 46)
     (tracks 602)
     (zones 0)
@@
     (pad_drill 0.762)
     (pad_to_mask_clearance 0.2)
-    (solder_mask_min_width 0.05)
     (aux_axis_origin 0 0)
     (visible_elements FFFFFF7F)
@@
     )
   )
+  (gr_text 1 (at 105.79 70.1) (layer B.SilkS)
+    (effects (font (size 0.8 0.8) (thickness 0.15)) (justify mirror))
+  )
   (gr_text - (at 165.5 88.75) (layer F.SilkS)
